Commit message: nav2 fixes

File: FollowBotAROS2/src/mapping/urdf/followbot.urdf.xacro (robot description, xacro)
@@ -58,5 +58,5 @@
       <material name="black">
         <color rgba="0 0 0 1"/>
-      </material>d
+      </material>
     </visual>
   </link>
@@ -64,5 +64,5 @@
     <parent link="base_link"/>
     <child link="left_wheel"/>
-    <origin xyz="0.15 0.2 -0.05" rpy="${pi/2} 0 0"/> <!-- position relative to base -->
+    <origin xyz="0.15 0.15 -0.05" rpy="${pi/2} 0 0"/> <!-- position relative to base -->
     <axis xyz="0 1 0"/> <!-- rotate around y-axis -->
   </joint>
@@ -79,5 +79,5 @@
     <parent link="base_link"/>
     <child link="right_wheel"/>
-    <origin xyz="0.15 -0.2 -0.05" rpy="${pi/2} 0 0"/> <!-- mirrored y-position -->
+    <origin xyz="0.15 -0.15 -0.05" rpy="${pi/2} 0 0"/> <!-- mirrored y-position -->
     <axis xyz="0 1 0"/>
   </joint>
@@ -97,5 +97,5 @@
     <child link="left_caster"/>
     <!-- positioned FORWARD on the left side (TODO: adjust x to robot's design) -->
-    <origin xyz="0.15 0.2 -0.05" rpy="0 0 0"/>
+    <origin xyz="-0.15 0.15 -0.05" rpy="0 0 0"/>
   </joint>
   <!-- Right Caster Wheel (passive, no encoder) -->
@@ -111,5 +111,5 @@
     <child link="right_caster"/>
     <!-- Positioned FORWARD on the right side -->
-    <origin xyz="0.15 -0.2 -0.05" rpy="0 0 0"/>
+    <origin xyz="-0.15 -0.15 -0.05" rpy="0 0 0"/>
   </joint>
 </robot>
